File: KiCad/FESS motor.kicad_sch (KiCad schematic)
At the start: 28 parts, among them J1 970KV BLDC Motor, J2 Hall effect sensor, J4 30A-ESC, J5 ACS712 hdr, J6 Motor (discharge), J7 ACS712 hdr #2

Commit message: Add files via upload
Parts:
- removed J5: ACS712 hdr, Connector:Tag-Connect_TC2030-IDC-FP_2x03_P1.27mm_Vertical, symbol Connector_Generic:Conn_01x03
- removed J7: ACS712 hdr #2, Connector:Tag-Connect_TC2030-IDC-FP_2x03_P1.27mm_Vertical, symbol Connector_Generic:Conn_01x03
- removed MES1: ACS712 IP+/IP-, symbol Device:Ammeter_DC
- removed MES2: ACS712 #2 IP+/IP-, symbol Device:Ammeter_DC
- added J6, J7: ACS712-30A-Ammeter, symbol Connector_Generic:Conn_01x05
- J3: renamed from J6; value Motor (discharge) -> 970KV BLDC Motor (Loc2)
Connections:
- net +5V: now also J6.Vcc (Pin_4), J7.Vcc (Pin_4)
- net GND: now also D8.2 (A), J6.GND (Pin_2), J6.IP- (Pin_5), J7.GND (Pin_2); no longer A1.10 (A1), D8.1 (K)
- net at D2.1 (K), D4.1 (K), D6.1 (K): now also J6.IP+ (Pin_1)
- net at A1.11 (A2), C2.2, R5.2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: now also D8.1 (K); no longer A1.12 (A3), A1.24 (D9), D8.2 (A), J4.SIGNAL (Pin_3)
- net at R1.1, Switch.2 (B): now also J7.IP+ (Pin_1)
- net at J4.BAT+ (Pin_1): now also J7.IP- (Pin_5)
- new net: A1.12 (A3), J6.VIout (Pin_3)
- new net: A1.24 (D9), J4.SIGNAL (Pin_3)
- new net: A1.10 (A1), J7.VIout (Pin_3)
Other:
- note added: "FESS Flywheel Project, Iteration 2"
- note removed: "FESS Flywheel Project, Iteration 1"
- moved on the sheet: A1, BT1, C1, C2, D1, D2, D3, D4, D5, D6, D7, D8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
